Commit message: adicionando material às peças que ainda não tinham

File: urdf_ws/src/robot_description/urdf/robot.urdf (robot description, URDF)
Before this commit: robot upper_body, 7 links, 6 joints
Links:
- link atom_braco: geometry collision mesh filename=assets/atom_braco.stl; collision mesh filename=assets/xm540.stl
- link atom_braco_2: geometry collision mesh filename=assets/atom_braco.stl; collision mesh filename=assets/xm540.stl
- link atom_mao: geometry collision mesh filename=assets/atom_mao.stl; collision mesh filename=assets/atom_mao.stl
- link atom_mao_2: geometry collision mesh filename=assets/atom_mao.stl; collision mesh filename=assets/atom_mao.stl
- link atom_ombro_chapa: geometry collision mesh filename=assets/atom_ombro.stl; collision mesh filename=assets/atom_ombro_chapa.stl
- link atom_ombro_chapa_2: geometry collision mesh filename=assets/atom_ombro.stl; collision mesh filename=assets/atom_ombro_chapa.stl
- link chest: geometry collision mesh filename=assets/atom_1_peito_frontal_impressao.stl; collision mesh filename=assets/atom_amortecedor_frente_corrigido.stl
